File: USemitter/Hardware/emitter.brd (EAGLE design)
At the start: 61.4 x 71.4 mm, 21 parts, among them U5 LM1117MP-3.3

Commit message: Final version of the emitter board
Parts:
- U$1, U$2: value MIC4605-2YM -> MIC4605-1YM
- moved U$1 2.68 mm to (15.7, 48.4)
- moved U$2 1.66 mm to (12.3, 12.1)
- moved C4 1.15 mm to (13.3, 56.6)
- moved C6 0.36 mm to (5.59, 12.6), turned to 90 degrees
Connections:
- net +9V: now also U$2.7; no longer U$2.1
- net GND: now also U$2.1; no longer U$2.7
- net N$9: now also U$2.4; no longer U$2.2
- net OUT2: now also U$2.2; no longer U$2.4
- net PWM: now also U$2.6
- net PWM/: now also U$1.6
Routing:
- net PWM: track 15.1 -> 63.2 mm, vias 0 -> 2
- net PWM/: track 16.3 -> 51.8 mm, vias 0 -> 2
- net GND: track 235.4 -> 253.6 mm, vias 6 -> 9
- net N$5: track 16.0 -> 24.2 mm, vias 0 -> 2
- net N$6: track 20.5 -> 27.9 mm, vias 0 -> 2
- net +9V: track 152.0 -> 157.1 mm, vias 3 -> 4
- net OUT1: track 47.6 -> 50.5 mm
- net N$7: track 4.25 -> 5.77 mm
- net N$4: track 6.53 -> 5.09 mm
- net N$3: track 13.3 -> 14.5 mm
- net OUT2: track 28.0 -> 29.0 mm
- net N$9: track 3.28 -> 4.13 mm
